File: Tiny433MHz/tiny433mhz.sch (EAGLE design)
At the start: 10 parts, among them U1 ATTINY85V-10SU

Commit message: updated WiSwitch, tiny433mhz and ade7953
Parts:
- removed C3: 10uF, rcl:C-EUC1206
- removed JP2: (no value), adafruit:PINHD-1X1
- removed SV3: (no value), con-lstb:MA03-1
- removed U1: ATTINY85V-10SU, atmel:ATTINY85V-10SU
- added LED1, LED2: (no value), adafruit:LEDCHIP-LED0805
- added R3: 10k, rcl:R-EU_R0805
- added U$1: ATTINY13SOIC, SparkFun:ATTINY13SOIC
- added U$3: CR2032, _CR2032:CR2032
- R2: value 4,7k -> 10k
Connections:
- removed net 1WIRE: R2.2, SV3.2, U1.PB3
- new net LED: LED2.C, U$1.PB3(ADC3)
- new net N$1: LED2.A, R3.2
- new net N$2: LED1.A, R2.2
- net DATA: now also SV1.1, U$1.PB4(ADC2); no longer SV1.3, U1.PB4
- net GND: now also R3.1, SV1.3, U$1.GND, U$3.-; no longer C3.2, SV1.1, SV3.1, U1.GND
- net MISO: now also U$1.PB1(MISO); no longer U1.PB1
- net MOSI: now also LED1.C, SV2.1, U$1.PB0(MOSI); no longer SV2.3, U1.PB0
- net RESET: now also U$1.PB5(NRES); no longer U1.PB5
- net SCK: now also SV2.3, U$1.PB2(SCK/ADC1); no longer SV2.1, U1.PB2
- net VCC: now also U$1.VCC, U$3.+; no longer C3.1, JP2.1, SV3.3, U1.VCC
Other:
- moved on the sheet: R2, SV1
