File: WiSwitch/WiSwitch.sch (EAGLE design)
At the start: 22 parts, among them IC1 REG1117, T1 BT136

Commit message: updated WiSwitch, tiny433mhz and ade7953
Parts:
- removed R8: (no value), rcl:R-EU_R0603
- added C4, C5: (no value), rcl:C-EUC0805
- added L1: WS2812B, adafruit:WS2812B
- added LED1: (no value), adafruit:LEDCHIP-LED0805
- added R10: 10k, rcl:R-EU_R0805
Connections:
- net N$6 renamed TX
- net N$7 renamed RX
- new net GPIO4: R10.2, X1.GPIO4
- new net GPIO5: U$3.OUT, X1.GPIO5
- new net N$7: LED1.A, R10.1
- net 5V: now also C5.2, L1.VDD
- net GND: now also C4.1, C5.1, L1.GND, LED1.C; no longer R8.2
- net GPIO0: no longer R8.1
- net GPIO13: now also L1.DIN; no longer R3.1
- net GPIO14: now also R3.1, X1.GPIO14; no longer U$3.OUT
- net VCC: now also C4.2
Other:
- moved on the sheet: R6
